File: ssc.kicad_sch (KiCad schematic)
At the start: 30 parts, among them J1 IRQ ENABLE, J2 RS-232 OUT, P1 A2Bus, U1 74LS245, U2 27C256, U3 1.8432M, U3 74HC00, U4 SSCGLU, U5 W65C51NxP, U6 MAX3232, U7 MAX3232, Y1 1.8432 MHz

Commit message: Checkpoint.
Connections:
- net A3: no longer U4.11 (A3)
- net D0: no longer U4.22 (D0)
- net R~{W}: no longer U4.6 (R~{W})
- net at U5.9 (~{CTS}), U6.9 (R2OUT): no longer U4.2 (CTS)
- no-connect marks 23 -> 27
Changed lines of the file:
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@@
 (kicad_sch (version 20230121) (generator eeschema)
   (paper "A3")
-  (junction (at 264.16 83.82) (diameter 0) (color 0 0 0 0)
-  )
   (junction (at 72.39 210.82) (diameter 0) (color 0 0 0 0)
   )
@@
   (no_connect (at 246.38 53.34))
   (no_connect (at 66.04 68.58))
+  (no_connect (at 168.91 205.74))
   (no_connect (at 66.04 60.96))
+  (no_connect (at 168.91 200.66))
+  (no_connect (at 168.91 220.98))
   (no_connect (at 66.04 86.36))
   (no_connect (at 66.04 88.9))
@@
   (no_connect (at 66.04 101.6))
   (no_connect (at 30.48 73.66))
+  (no_connect (at 203.2 222.25))
   (no_connect (at 66.04 93.98))
   (no_connect (at 50.8 116.84))
@@
     (stroke (width 0) (type default))
   )
-  (wire (pts (xy 203.2 222.25) (xy 210.82 222.25))
-    (stroke (width 0) (type default))
-  )
   (wire (pts (xy 72.39 210.82) (xy 72.39 223.52))
     (stroke (width 0) (type default))
@@
     (stroke (width 0) (type default))
   )
-  (wire (pts (xy 139.7 220.98) (xy 139.7 163.83))
-    (stroke (width 0) (type default))
-  )
   (wire (pts (xy 368.3 232.41) (xy 368.3 236.22))
     (stroke (width 0) (type default))
@@
     (stroke (width 0) (type default))
   )
-  (wire (pts (xy 168.91 205.74) (xy 161.29 205.74))
-    (stroke (width 0) (type default))
-  )
   (wire (pts (xy 210.82 88.9) (xy 215.9 88.9))
     (stroke (width 0) (type default))
@@
     (stroke (width 0) (type default))
   )
-  (wire (pts (xy 243.84 163.83) (xy 243.84 109.22))
-    (stroke (width 0) (type default))
-  )
   (wire (pts (xy 25.4 40.64) (xy 30.48 40.64))
     (stroke (width 0) (type default))
@@
     (stroke (width 0) (type default))
   )
-  (wire (pts (xy 264.16 83.82) (xy 264.16 109.22))
-    (stroke (width 0) (type default))
-  )
   (wire (pts (xy 186.69 238.76) (xy 186.69 241.3))
     (stroke (width 0) (type default))
@@
     (stroke (width 0) (type default))
   )
-  (wire (pts (xy 139.7 163.83) (xy 243.84 163.83))
-    (stroke (width 0) (type default))
-  )
   (wire (pts (xy 67.31 231.14) (xy 67.31 233.68))
     (stroke (width 0) (type default))
@@
     (stroke (width 0) (type default))
   )
-  (wire (pts (xy 139.7 220.98) (xy 168.91 220.98))
-    (stroke (width 0) (type default))
-  )
   (wire (pts (xy 135.89 100.33) (xy 128.27 100.33))
     (stroke (width 0) (type default))
@@
     (stroke (width 0) (type default))
   )
-  (wire (pts (xy 152.4 200.66) (xy 168.91 200.66))
-    (stroke (width 0) (type default))
-  )
   (wire (pts (xy 26.67 109.22) (xy 26.67 135.89))
     (stroke (width 0) (type default))
@@
     (stroke (width 0) (type default))
   )
-  (wire (pts (xy 243.84 109.22) (xy 264.16 109.22))
-    (stroke (width 0) (type default))
-  )
-  (global_label "R~{W}" (shape input) (at 152.4 200.66 180) (fields_autoplaced)
-    (effects (font (size 1.27 1.27)) (justify right))
-    (property "Intersheetrefs" "${INTERSHEET_REFS}" (at 147.427 200.66 0)
-      (effects (font (size 1.27 1.27)) (justify right) hide)
-    )
-  )
   (global_label "D5" (shape bidirectional) (at 161.29 95.25 0) (fields_autoplaced)
     (effects (font (size 1.27 1.27)) (justify left))
@@
     )
   )
-  (global_label "D0" (shape tri_state) (at 210.82 222.25 0) (fields_autoplaced)
-    (effects (font (size 1.27 1.27)) (justify left))
-    (property "Intersheetrefs" "${INTERSHEET_REFS}" (at 216.5036 222.25 0)
-      (effects (font (size 1.27 1.27)) (justify left) hide)
-    )
-  )
   (global_label "D1" (shape bidirectional) (at 33.02 176.53 180) (fields_autoplaced)
     (effects (font (size 1.27 1.27)) (justify right))
@@
       (effects (font (size 1.27 1.27)) (justify right) hide)
     )
-  )
-  (global_label "A3" (shape input) (at 161.29 205.74 180) (fields_autoplaced)
-    (effects (font (size 1.27 1.27)) (justify right))
-    (property "Intersheetrefs" "${INTERSHEET_REFS}" (at 156.7403 205.74 0)
-      (effects (font (size 1.27 1.27)) (justify right) hide)
-    )

Commit message: Checkpoint.
Parts:
- P1: symbol ssc-rescue:A2Bus-apple2 -> apple2:A2Bus
- U4: value SSCGLU -> GAL22V10D; symbol ssc:SSCGLU -> Logic_Programmable:PAL24
- U5: footprint Package_DIP:DIP-28_W15.24mm_Socket -> Package_DIP:DIP-28_W15.24mm; symbol ssc-rescue:W65C51NxP-65xx -> 65xx:6551
Connections:
- no-connect marks 27 -> 31
Other:
- moved on the sheet: J1

Commit message: Checkpoint.
Parts:
- C10, C11, C12, C13, C14, C15, C16, C9: symbol ssc-rescue:CP_Small-Device -> Device:C_Polarized_Small
- J1: symbol ssc-rescue:Conn_01x02_Male-Connector -> Connector:Conn_01x02_Pin
- J2: symbol ssc:Conn_PC_MB_Serial -> Connector:Conn_01x10_Pin
Connections:
- net SERCLK: no longer U3.8
- net RxD: now reaches J2.2 (Pin_2), U6.13 (R1IN)
- net TxD: now reaches J2.3 (Pin_3), U6.14 (T1OUT)
- net RTS: now reaches J2.7 (Pin_7), U6.7 (T2OUT)
- net CTS: now reaches J2.8 (Pin_8), U6.8 (R2IN)
- net DSR: now reaches J2.6 (Pin_6), U7.13 (R1IN)
- net DTR: now reaches J2.4 (Pin_4), U7.14 (T1OUT)
- net DCD: now reaches J2.1 (Pin_1), U7.8 (R2IN)
Other:
- note added: "RI"
Changed lines of the file:
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@@
   (no_connect (at 50.8 116.84))
   (no_connect (at 246.38 48.26))
-  (no_connect (at 360.68 109.22))
+  (no_connect (at 360.68 111.76))
   (no_connect (at 66.04 96.52))
   (no_connect (at 66.04 91.44))
@@
   (no_connect (at 66.04 66.04))
   (no_connect (at 313.69 153.67))
-  (no_connect (at 115.824 226.06))
+  (no_connect (at 360.68 114.3))
   (no_connect (at 201.93 205.74))
   (wire (pts (xy 66.04 53.34) (xy 73.66 53.34))
@@
     (stroke (width 0) (type default))
   )
-  (wire (pts (xy 204.978 55.88) (xy 196.088 55.88))
+  (wire (pts (xy 195.834 55.88) (xy 204.978 55.88))
     (stroke (width 0) (type default))
   )
@@
     (stroke (width 0) (type default))
   )
+  (wire (pts (xy 360.68 101.6) (xy 351.79 101.6))
+    (stroke (width 0) (type default))
+  )
   (wire (pts (xy 25.4 40.64) (xy 30.48 40.64))
     (stroke (width 0) (type default))
@@
     (stroke (width 0) (type default))
   )
-  (wire (pts (xy 360.68 101.6) (xy 340.36 101.6))
+  (wire (pts (xy 360.68 104.14) (xy 340.36 104.14))
     (stroke (width 0) (type default))
   )
@@
     (stroke (width 0) (type default))
   )
-  (wire (pts (xy 336.55 104.14) (xy 360.68 104.14))
+  (wire (pts (xy 336.55 106.68) (xy 360.68 106.68))
     (stroke (width 0) (type default))
   )
@@
     (stroke (width 0) (type default))
   )
-  (wire (pts (xy 328.93 106.68) (xy 328.93 83.82))
+  (wire (pts (xy 328.93 109.22) (xy 328.93 83.82))
     (stroke (width 0) (type default))
   )
@@
     (stroke (width 0) (type default))
   )
-  (wire (pts (xy 360.68 106.68) (xy 328.93 106.68))
+  (wire (pts (xy 360.68 109.22) (xy 328.93 109.22))
     (stroke (width 0) (type default))
   )
@@
     (stroke (width 0) (type default))
   )
-  (wire (pts (xy 368.3 121.92) (xy 368.3 123.19))
+  (wire (pts (xy 351.79 101.6) (xy 351.79 112.014))
     (stroke (width 0) (type default))
   )
@@
     (stroke (width 0) (type default))
   )
-  (wire (pts (xy 336.55 73.66) (xy 336.55 104.14))
+  (wire (pts (xy 336.55 73.66) (xy 336.55 106.68))
     (stroke (width 0) (type default))
   )
@@
     (stroke (width 0) (type default))
   )
-  (wire (pts (xy 340.36 101.6) (xy 340.36 158.75))
+  (wire (pts (xy 340.36 104.14) (xy 340.36 158.75))
     (stroke (width 0) (type default))
   )
@@
     (stroke (width 0) (type default))
   )
-  (wire (pts (xy 196.088 53.34) (xy 215.9 53.34))
+  (wire (pts (xy 195.834 53.34) (xy 215.9 53.34))
     (stroke (width 0) (type default))
   )
@@
     (stroke (width 0) (type default))
   )
+  (text "RI" (at 355.854 111.76 0)
+    (effects (font (size 1.27 1.27)) (justify left bottom))
+  )
+  (label "DCD" (at 356.362 91.44 0) (fields_autoplaced)
+    (effects (font (size 1.27 1.27)) (justify left bottom))
+  )
+  (label "DTR" (at 355.854 99.06 0) (fields_autoplaced)
+    (effects (font (size 1.27 1.27)) (justify left bottom))
+  )
+  (label "DSR" (at 355.854 104.14 0) (fields_autoplaced)
+    (effects (font (size 1.27 1.27)) (justify left bottom))
+  )
+  (label "CTS" (at 355.6 109.22 0) (fields_autoplaced)
+    (effects (font (size 1.27 1.27)) (justify left bottom))
+  )
+  (label "RTS" (at 355.854 106.68 0) (fields_autoplaced)
+    (effects (font (size 1.27 1.27)) (justify left bottom))
+  )
+  (label "RxD" (at 356.362 93.98 0) (fields_autoplaced)
+    (effects (font (size 1.27 1.27)) (justify left bottom))
+  )
+  (label "TxD" (at 356.108 96.52 0) (fields_autoplaced)
+    (effects (font (size 1.27 1.27)) (justify left bottom))
+  )
   (global_label "D5" (shape bidirectional) (at 161.29 95.25 0) (fields_autoplaced)
     (effects (font (size 1.27 1.27)) (justify left))
@@
     (property "Intersheetrefs" "${INTERSHEET_REFS}" (at 156.6799 200.66 0)
       (effects (font (size 1.27 1.27)) (justify right) hide)
-    )
-  )
-  (global_label "SERCLK" (shape input) (at 125.73 208.28 0) (fields_autoplaced)
-    (effects (font (size 1.27 1.27)) (justify left))
-    (property "Intersheetrefs" "${INTERSHEET_REFS}" (at 135.1782 208.28 0)
-      (effects (font (size 1.27 1.27)) (justify left) hide)
     )
   )
@@
     )
   )
-  (symbol (lib_id "ssc-rescue:CP_Small-Device") (at 266.7 46.99 0) (mirror y) (unit 1)
+  (symbol (lib_id "Device:C_Polarized_Small") (at 266.7 46.99 0) (mirror y) (unit 1)
     (in_bom yes) (on_board yes) (dnp no)
     (property "Reference" "C9" (at 269.0368 45.8216 0)
@@
     )
   )
-  (symbol (lib_id "ssc-rescue:CP_Small-Device") (at 320.04 46.99 0) (unit 1)
+  (symbol (lib_id "Device:C_Polarized_Small") (at 320.04 46.99 0) (unit 1)
     (in_bom yes) (on_board yes) (dnp no)
     (property "Reference" "C11" (at 317.7032 45.8216 0)
@@
     )
   )
-  (symbol (lib_id "ssc-rescue:CP_Small-Device") (at 372.11 55.88 90) (unit 1)
+  (symbol (lib_id "Device:C_Polarized_Small") (at 372.11 55.88 90) (unit 1)
     (in_bom yes) (on_board yes) (dnp no)
     (property "Reference" "C15" (at 370.84 54.61 90)
@@
     )
   )
-  (symbol (lib_id "ssc-rescue:CP_Small-Device") (at 372.11 63.5 270) (unit 1)
+  (symbol (lib_id "Device:C_Polarized_Small") (at 372.11 63.5 270) (unit 1)
     (in_bom yes) (on_board yes) (dnp no)
     (property "Reference" "C13" (at 367.03 62.23 90)
@@
     )
   )
-  (symbol (lib_id "ssc-rescue:CP_Small-Device") (at 266.7 127 0) (mirror y) (unit 1)
+  (symbol (lib_id "Device:C_Polarized_Small") (at 266.7 127 0) (mirror y) (unit 1)
     (in_bom yes) (on_board yes) (dnp no)
     (property "Reference" "C10" (at 269.0368 125.8316 0)
@@
     )
   )
-  (symbol (lib_id "ssc-rescue:Conn_01x02_Male-Connector") (at 191.008 53.34 0) (unit 1)
-    (in_bom yes) (on_board yes) (dnp no)
-    (property "Reference" "J1" (at 193.7512 48.7426 0)
-      (effects (font (size 1.27 1.27)))
-    )
-    (property "Value" "IRQ ENABLE" (at 193.7512 51.054 0)
-      (effects (font (size 1.27 1.27)))
-    )
-    (property "Footprint" "Connector_PinHeader_2.54mm:PinHeader_1x02_P2.54mm_Vertical" (at 191.008 53.34 0)
-      (effects (font (size 1.27 1.27)) hide)
-    )
-    (property "Datasheet" "~" (at 191.008 53.34 0)
+  (symbol (lib_id "Connector:Conn_01x02_Pin") (at 190.754 53.34 0) (unit 1)
+    (in_bom yes) (on_board yes) (dnp no)
+    (property "Reference" "J1" (at 193.4972 48.7426 0)
+      (effects (font (size 1.27 1.27)))
+    )
+    (property "Value" "IRQ ENABLE" (at 193.4972 51.054 0)
+      (effects (font (size 1.27 1.27)))
+    )
+    (property "Footprint" "Connector_PinHeader_2.54mm:PinHeader_1x02_P2.54mm_Vertical" (at 190.754 53.34 0)
+      (effects (font (size 1.27 1.27)) hide)
+    )
+    (property "Datasheet" "~" (at 190.754 53.34 0)
       (effects (font (size 1.27 1.27)) hide)
     )
@@
     )
   )
-  (symbol (lib_id "ssc-rescue:CP_Small-Device") (at 320.04 127 0) (unit 1)
+  (symbol (lib_id "Device:C_Polarized_Small") (at 320.04 127 0) (unit 1)
     (in_bom yes) (on_board yes) (dnp no)
     (property "Reference" "C12" (at 317.7032 125.8316 0)
@@
     )
   )
-  (symbol (lib_id "ssc-rescue:CP_Small-Device") (at 372.11 135.89 90) (unit 1)
+  (symbol (lib_id "Device:C_Polarized_Small") (at 372.11 135.89 90) (unit 1)
     (in_bom yes) (on_board yes) (dnp no)
     (property "Reference" "C16" (at 370.84 134.62 90)
@@
     )
   )
-  (symbol (lib_id "ssc-rescue:CP_Small-Device") (at 372.11 143.51 270) (unit 1)
+  (symbol (lib_id "Device:C_Polarized_Small") (at 372.11 143.51 270) (unit 1)
     (in_bom yes) (on_board yes) (dnp no)
     (property "Reference" "C14" (at 367.03 142.24 90)
@@
     )
   )
-  (symbol (lib_id "ssc:Conn_PC_MB_Serial") (at 368.3 104.14 0) (unit 1)
-    (in_bom yes) (on_board yes) (dnp no)
-    (property "Reference" "J2" (at 368.3 85.09 0)
-      (effects (font (size 1.27 1.27)))
-    )
-    (property "Value" "RS-232 OUT" (at 368.3 87.63 0)
-      (effects (font (size 1.27 1.27)))
-    )
-    (property "Footprint" "Connector_PinHeader_2.54mm:PinHeader_2x05_P2.54mm_Vertical" (at 368.3 104.14 0)
-      (effects (font (size 1.27 1.27)) hide)
-    )
-    (property "Datasheet" "" (at 368.3 104.14 0)
-      (effects (font (size 1.27 1.27)) hide)
-    )
-    (pin "1")
+  (symbol (lib_id "Connector:Conn_01x10_Pin") (at 365.76 101.6 0) (mirror y) (unit 1)
+    (in_bom yes) (on_board yes) (dnp no)
+    (property "Reference" "J2" (at 365.76 82.55 0)
+      (effects (font (size 1.27 1.27)))
+    )
+    (property "Value" "RS-232 OUT" (at 365.76 85.09 0)
+      (effects (font (size 1.27 1.27)))
+    )
+    (property "Footprint" "Connector_PinHeader_2.54mm:PinHeader_2x05_P2.54mm_Vertical" (at 365.76 101.6 0)
+      (effects (font (size 1.27 1.27)) hide)
+    )
+    (property "Datasheet" "~" (at 365.76 101.6 0)
+      (effects (font (size 1.27 1.27)) hide)
+    )
+    (pin "1")
+    (pin "10")
     (pin "2")
     (pin "3")
@@
     )
   )
-  (symbol (lib_id "power:GND") (at 368.3 123.19 0) (unit 1)
-    (in_bom yes) (on_board yes) (dnp no)
-    (property "Reference" "#PWR0118" (at 368.3 129.54 0)
-      (effects (font (size 1.27 1.27)) hide)
-    )
-    (property "Value" "GND" (at 368.427 127.5842 0)
-      (effects (font (size 1.27 1.27)))
-    )
-    (property "Footprint" "" (at 368.3 123.19 0)
-      (effects (font (size 1.27 1.27)) hide)
-    )
-    (property "Datasheet" "" (at 368.3 123.19 0)
-      (effects (font (size 1.27 1.27)) hide)
-    )
+  (symbol (lib_id "power:GND") (at 351.79 112.014 0) (unit 1)
+    (in_bom yes) (on_board yes) (dnp no)
+    (property "Reference" "#PWR0118" (at 351.79 118.364 0)
+      (effects (font (size 1.27 1.27)) hide)
+    )
+    (property "Value" "GND" (at 351.917 116.4082 0)
+      (effects (font (size 1.27 1.27)))
+    )
+    (property "Footprint" "" (at 351.79 112.014 0)
+      (effects (font (size 1.27 1.27)) hide)
+    )
+    (property "Datasheet" "" (at 351.79 112.014 0)
+      (effects (font (size 1.27 1.27)) hide)
+    )

Commit message: Checkpoint.
Parts:
- removed C17, C8: 20 pF, Capacitor_THT:C_Disc_D4.3mm_W1.9mm_P5.00mm, symbol Device:C_Small
- removed R1: 1M, Resistor_THT:R_Axial_DIN0207_L6.3mm_D2.5mm_P7.62mm_Horizontal, symbol Device:R
- removed unit 5 of U3
- removed unit 4 of U3
- removed unit 2 of U3
- removed unit 3 of U3
- removed Y1: 1.8432 MHz, Crystal:Crystal_HC49-U_Vertical, symbol Device:Crystal
- U3: value 1.8432M -> 1.8432 MHz
- U5: value W65C51NxP -> 6551
- U6, U7: value MAX3232 -> MAX232; symbol Interface_UART:MAX3232 -> Interface_UART:MAX232
Other:
- moved on the sheet: C1, C10, C11, C12, C13, C14, C15, C16, C2, C3, C4, C5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
